File: cnc_heat.kicad_sch (KiCad schematic)
At the start: 55 parts, among them J1 Raspberry_Pi_2_3, J2 DB25_Receptacle_MountingHoles, U1 74LVC1T45, U10 74LVC1T45, U11 74LVC1T45, U12 74LVC1T45, U13 74LVC1T45, U14 74LVC1T45, U15 74LVC1T45, U16 74LVC1T45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

Commit message: ocd routing
Parts:
- renumbered C5 to C4, C6 to C5, C7 to C6
Changed lines of the file:
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@@
 		(dnp no)
 		(fields_autoplaced yes)
-		(property "Reference" "C6"
+		(property "Reference" "C5"
 			(at 250.19 148.5899 0)
 			(effects
@@
 			(project "cnc_heat"
 				(path "/58fa3ba6-f076-4451-8045-d6c44cdcfd4b"
-					(reference "C6")
+					(reference "C5")
 					(unit 1)
 				)
@@
 		(dnp no)
 		(fields_autoplaced yes)
-		(property "Reference" "C5"
+		(property "Reference" "C4"
 			(at 237.49 148.5899 0)
 			(effects
@@
 			(project "cnc_heat"
 				(path "/58fa3ba6-f076-4451-8045-d6c44cdcfd4b"
-					(reference "C5")
+					(reference "C4")
 					(unit 1)
 				)
@@
 		(dnp no)
 		(fields_autoplaced yes)
-		(property "Reference" "C7"
+		(property "Reference" "C6"
 			(at 262.89 148.5899 0)
 			(effects
@@
 			(project "cnc_heat"
 				(path "/58fa3ba6-f076-4451-8045-d6c44cdcfd4b"
-					(reference "C7")
+					(reference "C6")
 					(unit 1)
 				)

Commit message: ocd routing
Parts:
- renumbered C4 to C1, C1 to C2, C5 to C3, C2 to C4, C6 to C5, C3 to C6
Changed lines of the file:
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@@
 		(dnp no)
 		(fields_autoplaced yes)
-		(property "Reference" "C1"
+		(property "Reference" "C2"
 			(at 237.49 133.3499 0)
 			(effects
@@
 			(project "cnc_heat"
 				(path "/58fa3ba6-f076-4451-8045-d6c44cdcfd4b"
-					(reference "C1")
+					(reference "C2")
 					(unit 1)
 				)
@@
 		(dnp no)
 		(fields_autoplaced yes)
-		(property "Reference" "C5"
+		(property "Reference" "C3"
 			(at 250.19 148.5899 0)
 			(effects
@@
 			(project "cnc_heat"
 				(path "/58fa3ba6-f076-4451-8045-d6c44cdcfd4b"
-					(reference "C5")
+					(reference "C3")
 					(unit 1)
 				)
@@
 		(dnp no)
 		(fields_autoplaced yes)
-		(property "Reference" "C2"
+		(property "Reference" "C4"
 			(at 250.19 133.3499 0)
 			(effects
@@
 			(project "cnc_heat"
 				(path "/58fa3ba6-f076-4451-8045-d6c44cdcfd4b"
-					(reference "C2")
+					(reference "C4")
 					(unit 1)
 				)
@@
 		(dnp no)
 		(fields_autoplaced yes)
-		(property "Reference" "C3"
+		(property "Reference" "C6"
 			(at 262.89 133.3499 0)
 			(effects
@@
 			(project "cnc_heat"
 				(path "/58fa3ba6-f076-4451-8045-d6c44cdcfd4b"
-					(reference "C3")
+					(reference "C6")
 					(unit 1)
 				)
@@
 		(dnp no)
 		(fields_autoplaced yes)
-		(property "Reference" "C4"
+		(property "Reference" "C1"
 			(at 237.49 148.5899 0)
 			(effects
@@
 			(project "cnc_heat"
 				(path "/58fa3ba6-f076-4451-8045-d6c44cdcfd4b"
-					(reference "C4")
+					(reference "C1")
 					(unit 1)
 				)
@@
 		(dnp no)
 		(fields_autoplaced yes)
-		(property "Reference" "C6"
+		(property "Reference" "C5"
 			(at 262.89 148.5899 0)
 			(effects
@@
 			(project "cnc_heat"
 				(path "/58fa3ba6-f076-4451-8045-d6c44cdcfd4b"
-					(reference "C6")
+					(reference "C5")
 					(unit 1)
 				)
